File: first kicadfile.kicad_sch (KiCad schematic)
At the start: 14 parts

Commit message: Final version
lol i forgot to use github but this should be all the kicad files i used, as well as the final gerber and cut files
Parts:
- added D1, D2, D3, D4: D_Small, Diode_SMD:D_SOD-123, symbol Device:D_Small
- added F1: 500mA, Fuse:Fuse_1206_3216Metric, symbol Device:Polyfuse
- added MX1, MX2, MX3, MX4: MX-NoLED, MX_Alps_Hybrid:MX-1U-NoLED, symbol MX_Alps_Hybrid:MX-NoLED
- added SW2: RotaryEncoder_Switch, Rotary_Encoder:RotaryEncoder_Alps_EC11E-Switch_Vertical_H20mm_CircularMountingHoles, symbol Device:RotaryEncoder_Switch
- added USB1: Molex-0548190589, random-keyboard-parts:Molex-0548190589, symbol random-keyboard-parts:Molex-0548190589
- C1, C2, C3, C4, C5, C6, C7: renamed from C?; footprint (none) -> Capacitor_SMD:C_0805_2012Metric
- R1, R2, R3, R4: renamed from R?; footprint (none) -> Resistor_SMD:R_0805_2012Metric
- SW1: renamed from SW?; footprint (none) -> random-keyboard-parts:SKQG-1155865
- Y1: renamed from Y?; footprint (none) -> Crystal:Crystal_SMD_3225-4Pin_3.2x2.5mm
- gave numbers to parts that had none: 1
Connections:
- net +5V: now also F1.2
- net D+: now also USB1.3 (D+)
- net D-: now also USB1.4 (D-)
- net GND: now also USB1.1 (GND)
- net PB2: now reaches U1.10 (PB2)
- net PB2: now also SW2.B
- net PB7: now reaches U1.12 (PB7)
- net PB7: now also SW2.S2
- net ROW0: now reaches U1.28 (PB4)
- net ROW0: now also D1.1 (K), D3.1 (K)
- net ROW1: now reaches U1.29 (PB5)
- net ROW1: now also D2.1 (K), D4.1 (K)
- net PB6: now reaches U1.30 (PB6)
- net PB6: now also SW2.S1
- net COL0: now reaches U1.36 (PF7)
- net COL0: now also MX1.1 (COL), MX2.1 (COL)
- net COL1: now reaches U1.37 (PF6)
- net COL1: now also MX3.1 (COL), MX4.1 (COL)
- net PB0: now reaches U1.8 (PB0)
- net PB0: now also SW2.A
- net PB1: now reaches U1.9 (PB1)
- net PB1: now also SW2.C
- new net: D3.2 (A), MX3.2 (ROW)
- new net: D1.2 (A), MX1.2 (ROW)
- new net: D2.2 (A), MX2.2 (ROW)
- new net: D4.2 (A), MX4.2 (ROW)
- new net VCC: F1.1, USB1.5 (VBUS)
Other:
- moved on the sheet: C1, C2, C3, C4, C5, C6, C7, R1, R2, R3, R4, SW1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
